File: Merax Wiring/Merax Wiring.sch (KiCad schematic (older format))
At the start: 54 parts

Commit message: Corrected wiring schematic (use Eeschema to view)
Parts:
- removed J?: Com_Cable, symbol Merax_EBike_Parts:Com_Cable
- added J?: AudioJack2_Ground, symbol Connector:AudioJack2_Ground
- added J?: XLR3_AudioJack2_Combo, symbol Connector:XLR3_AudioJack2_Combo
Connections:
- net at U?.2 (3V3): now also U?.2 (OUT)
- net at U?.26 (IO4): now also U?.34 (RXD0), U?.~, J?.1, J?.T
- net at U?.~: now also J?.2, J?.S
- net at U?.~ (yellow): now also BT?.1 (+), U?.1 (VIN), U?.~ (Power); no longer U?.~ (y)
- net at U?.~ (y): now also J?.6 (Hall); no longer U?.~ (yellow)
- net at J?.1 (Pin_1), J?.1 (Pin_1), J?.1 (Pin_1): no longer J?.1 (Pin_1)
- net at J?.1 (Pin_1), U?.~ (yellow): now also J?.1 (Pin_1)
- net at J?.2 (Pin_2), U?.~ (yellow): now also J?.2 (Pin_2)
- net at J?.2 (Pin_2), J?.2 (Pin_2): no longer J?.2 (Pin_2)
- new net: U?.~ (y), U?.~ (yellow) (x3)
- new net: J?.3, J?.G, U?.~
Other:
- note removed: "black"
- note removed: "blue"
- note removed: "green"
- note removed: "red"
- note removed: "white"
- note removed: "yellow"
